Commit message: urdf changes

File: unicorn_description/urdf/rplidar_a2.urdf.xacro (robot description, xacro)
@@ -10,5 +10,5 @@
 	    </inertial>
 	    <visual>
-		<origin xyz = "0.0 0.0 0.0" rpy= "0.0 0.0 0.0" />
+		<origin xyz = "0.0 0.0 0.28" rpy= "0.0 0.0 0.0" />
    	    </visual>
 	    <collision>

File: unicorn_description/urdf/unicorn_target.urdf.xacro (robot description, xacro)
@@ -6,7 +6,7 @@
   <property name="M_PI" value="3.1415926535897931" />
   <!-- Main Body-base -->
-  <property name="base_x_size" value="0.72" />
-  <property name="base_y_size" value="0.55" />
-  <property name="base_z_size" value="0.6" />
+  <property name="base_x_size" value="0.70" />
+  <property name="base_y_size" value="0.49" />
+  <property name="base_z_size" value="0.44" />
   <property name="base_mass" value="15" /> <!-- 21.446 in kg-->
   <!--Inertial macros for the box and cylinder. Units are kg*m^2-->
@@ -23,7 +23,8 @@
 -->
   <!-- Ultrasonic sensor -->
-  <xacro:arg name="ultrasonic_xyz" default="-0.3 0 0.2" />
+<!--  <xacro:arg name="ultrasonic_xyz" default="-0.3 0 0.2" />
   <xacro:arg name="ultrasonic_rpy" default="0 0 0" />
   <xacro:include filename="$(find unicorn_description)/urdf/ultrasonic_sensor.urdf.xacro" />
+-->
   <!-- RPLIDAR A2 -->
   <xacro:arg name="laser_xyz" default="0.0 0.0 0.5" />
@@ -234,4 +235,5 @@
   <swivel_wheel fb="front" lr="left" parent="chassis_link" translateY="-0.16" translateX="0.355" translateZ="0.03" wheel_radius="0.05" wheel_height="0.05" flip="0"/>
   <swivel_wheel fb="front" lr="right" parent="chassis_link" translateY="0.16" translateX="0.355" translateZ="0.03" wheel_radius="0.05" wheel_height="0.05" flip="0"/>
+ <!--
   <ultrasonic_sensor frame="base_ultrasonic_br" topic="br" robot_namespace="$(arg robot_namespace)"/>
   <joint name="ultrasonic_mount_joint_br" type="fixed">
@@ -282,4 +284,5 @@
     <child link="base_ultrasonic_fml" />
   </joint>
+-->
 <!-- NOT USED ANYMORE SINCE CHANGE OF LIDAR -->
   <!--  <sick_lms1xx frame="base_laser" topic="scan" robot_namespace="$(arg robot_namespace)"/>

Commit message: Applied fix on xarco files

File: unicorn_description/urdf/rplidar_a2.urdf.xacro (robot description, xacro)
@@ -7,5 +7,5 @@
 		<mass value="0.564" />
 		<origin xyz ="0 0 0" />
-		<inertia ixx ="0.003881243" ixy="0.0" ixz="0.0"							 iyy="0.000498940"  iyz="0.0"								 izz="0.003879257" />
+		<inertia ixx ="0.003881243" ixy="0.0" ixz="0.0"							 iyy="0.000498940"  iyz="0.0" izz="0.003879257" />
 	    </inertial>
 	    <visual>

File: unicorn_description/urdf/ultrasonic_sensor.urdf.xacro (robot description, xacro)
@@ -1,4 +1,4 @@
 <?xml version="1.0"?>
-<robot xmlns:xacro="http://ros.org/wiki/xacro">
+<robot xmlns:xacro="http://www.ros.org/wiki/xacro">
   <xacro:macro name="ultrasonic_sensor" params="frame topic:=sonar robot_namespace:=/" >
     <link name="${frame}">

File: unicorn_description/urdf/unicorn_cam.urdf.xacro (robot description, xacro)
@@ -19,17 +19,17 @@
   <!-- PROPERTY LIST -->
   <!--All units in m-kg-s-radians unit system -->
-  <property name="M_PI" value="3.1415926535897931" />
+  <xacro:property name="M_PI" value="3.1415926535897931" />
   <!-- Main Body-base -->
-  <property name="base_x_size" value="0.72" />
-  <property name="base_y_size" value="0.55" />
-  <property name="base_z_size" value="0.23" />
-  <property name="base_mass" value="15" /> <!-- in kg-->
-  <property name="base_z_origin_to_wheel_origin" value="-0.07" />
+  <xacro:property name="base_x_size" value="0.72" />
+  <xacro:property name="base_y_size" value="0.55" />
+  <xacro:property name="base_z_size" value="0.23" />
+  <xacro:property name="base_mass" value="15" /> <!-- in kg-->
+  <xacro:property name="base_z_origin_to_wheel_origin" value="-0.07" />
   <!--Inertial macros for the box and cylinder. Units are kg*m^2-->
-  <macro name="box_inertia" params="m x y z">
+  <xacro:macro name="box_inertia" params="m x y z">
     <inertia  ixx="${m*(y*y+z*z)/12}" ixy = "0" ixz = "0"
               iyy="${m*(x*x+z*z)/12}" iyz = "0"
               izz="${m*(x*x+z*z)/12}" />
-  </macro>
+  </xacro:macro>
   <!-- BASE-LINK -->
   <!--Actual body/chassis of the robot-->

File: unicorn_description/urdf/unicorn_sim.urdf.xacro (robot description, xacro)
@@ -4,16 +4,16 @@
   <xacro:arg name="robot_namespace" default="/" />
   <!--All units in m-kg-s-radians unit system -->
-  <property name="M_PI" value="3.1415926535897931" />
+  <xacro:property name="M_PI" value="3.1415926535897931" />
   <!-- Main Body-base -->
-  <property name="base_x_size" value="0.72" />
-  <property name="base_y_size" value="0.55" />
-  <property name="base_z_size" value="0.6" />
-  <property name="base_mass" value="15" /> <!-- 21.446 in kg-->
+  <xacro:property name="base_x_size" value="0.72" />
+  <xacro:property name="base_y_size" value="0.55" />
+  <xacro:property name="base_z_size" value="0.6" />
+  <xacro:property name="base_mass" value="15" /> <!-- 21.446 in kg-->
   <!--Inertial macros for the box and cylinder. Units are kg*m^2-->
-  <macro name="box_inertia" params="m x y z">
+  <xacro:macro name="box_inertia" params="m x y z">
     <inertia  ixx="${m*(y*y+z*z)/12}" ixy = "0" ixz = "0"
               iyy="${m*(x*x+z*z)/12}" iyz = "0"
               izz="${m*(x*x+z*z)/12}" />
-  </macro>
+  </xacro:macro>
   <!-- LMS111 -->
   <xacro:arg name="laser_xyz" default="0.0 0.0 0.260" />

File: unicorn_description/urdf/unicorn_target.urdf.xacro (robot description, xacro)
@@ -4,16 +4,16 @@
   <xacro:arg name="robot_namespace" default="/" />
   <!--All units in m-kg-s-radians unit system -->
-  <property name="M_PI" value="3.1415926535897931" />
+  <xacro:property name="M_PI" value="3.1415926535897931" />
   <!-- Main Body-base -->
-  <property name="base_x_size" value="0.70" />
-  <property name="base_y_size" value="0.49" />
-  <property name="base_z_size" value="0.44" />
-  <property name="base_mass" value="15" /> <!-- 21.446 in kg-->
+  <xacro:property name="base_x_size" value="0.70" />
+  <xacro:property name="base_y_size" value="0.49" />
+  <xacro:property name="base_z_size" value="0.44" />
+  <xacro:property name="base_mass" value="15" /> <!-- 21.446 in kg-->
   <!--Inertial macros for the box and cylinder. Units are kg*m^2-->
-  <macro name="box_inertia" params="m x y z">
+  <xacro:macro name="box_inertia" params="m x y z">
     <inertia  ixx="${m*(y*y+z*z)/12}" ixy = "0" ixz = "0"
               iyy="${m*(x*x+z*z)/12}" iyz = "0"
               izz="${m*(x*x+z*z)/12}" />
-  </macro>
+  </xacro:macro>
 <!-- NOT USED ANYMORE SINCE CHANGE OR LIDAR -->
   <!-- LMS111 -->
