Commit message: added RPlidar urdf

File: unicorn_description/urdf/unicorn_target.urdf.xacro (robot description, xacro)
@@ -16,12 +16,18 @@
               izz="${m*(x*x+z*z)/12}" />
   </macro>
+<!-- NOT USED ANYMORE SINCE CHANGE OR LIDAR -->
   <!-- LMS111 -->
-  <xacro:arg name="laser_xyz" default="0.0 0.0 0.5" />
+<!--  <xacro:arg name="laser_xyz" default="0.0 0.0 0.5" />
   <xacro:arg name="laser_rpy" default="0.0 0.0 ${M_PI-M_PI/4}" />
   <xacro:include filename="$(find lms1xx)/urdf/sick_lms1xx.urdf.xacro" />
+-->
   <!-- Ultrasonic sensor -->
   <xacro:arg name="ultrasonic_xyz" default="-0.3 0 0.2" />
   <xacro:arg name="ultrasonic_rpy" default="0 0 0" />
   <xacro:include filename="$(find unicorn_description)/urdf/ultrasonic_sensor.urdf.xacro" />
+  <!-- RPLIDAR A2 -->
+  <xacro:arg name="laser_xyz" default="0.0 0.0 0.5" />
+  <xacro:arg name="laser_rpy" default="0.0 0.0 ${M_PI-M_PI/4}" />
+  <xacro:include filename="$(find unicorn_description)/urdf/rplidar_a2.urdf.xacro" />
   <!-- Wheel -->
   <xacro:include filename="$(find am_description)/urdf/wheel.urdf.xacro" />
@@ -276,5 +282,6 @@
     <child link="base_ultrasonic_fml" />
   </joint>
-    <sick_lms1xx frame="base_laser" topic="scan" robot_namespace="$(arg robot_namespace)"/>
+<!-- NOT USED ANYMORE SINCE CHANGE OF LIDAR -->
+  <!--  <sick_lms1xx frame="base_laser" topic="scan" robot_namespace="$(arg robot_namespace)"/>
     <joint name="laser_mount_joint" type="fixed">
       <origin xyz="$(arg laser_xyz)" rpy="$(arg laser_rpy)" />
@@ -282,4 +289,11 @@
       <child link="base_laser" />
     </joint>
+-->
+   <rplidar_a2 frame="base_laser" topic="scan" robot_namespace="$(arg robot_namespace)"/>
+   <joint name="laser_mount_joint" type="fixed">
+      <origin xyz="$(arg laser_xyz)" rpy="$(arg laser_rpy)" />
+      <parent link="chassis_link" />
+      <child link="base_laser" />
+   </joint>
   <!-- GAZEBO STUFF -->
   <gazebo>

Commit message: new map and fixes

File: unicorn_description/urdf/unicorn_target.urdf.xacro (robot description, xacro)
@@ -27,5 +27,5 @@
   <xacro:include filename="$(find unicorn_description)/urdf/ultrasonic_sensor.urdf.xacro" />
   <!-- RPLIDAR A2 -->
-  <xacro:arg name="laser_xyz" default="0.0 0.0 0.5" />
+  <xacro:arg name="laser_xyz" default="0.15 0.0 0.5" />
   <xacro:arg name="laser_rpy" default="0.0 0.0 ${M_PI}" />
   <xacro:include filename="$(find unicorn_description)/urdf/rplidar_a2.urdf.xacro" />
@@ -236,5 +236,5 @@
   <ultrasonic_sensor frame="base_ultrasonic_br" topic="br" robot_namespace="$(arg robot_namespace)"/>
   <joint name="ultrasonic_mount_joint_br" type="fixed">
-    <origin xyz="0.45 0.2 0.0" rpy="0 0 ${3*M_PI/4}"/>
+    <origin xyz="0.45 0.1 0.0" rpy="0 0 0"/>
     <parent link="chassis_link"/>
     <child link="base_ultrasonic_br" />
@@ -242,5 +242,5 @@
   <ultrasonic_sensor frame="base_ultrasonic_bl" topic="bl" robot_namespace="$(arg robot_namespace)"/>
   <joint name="ultrasonic_mount_joint_bl" type="fixed">
-    <origin xyz="0.45 -0.2 0.0" rpy="0 0 ${M_PI-55*M_PI/180}"/>
+    <origin xyz="0.45 -0.1 0.0" rpy="0 0 0"/>
     <parent link="chassis_link"/>
     <child link="base_ultrasonic_bl" />

Commit message: Moved lidar and zed tf to correct prosition

File: unicorn_description/urdf/unicorn_target.urdf.xacro (robot description, xacro)
@@ -27,6 +27,8 @@
   <xacro:include filename="$(find unicorn_description)/urdf/ultrasonic_sensor.urdf.xacro" />
   <!-- RPLIDAR A2 -->
-  <xacro:arg name="laser_xyz" default="0.18 0.12 0.39" />
-  <xacro:arg name="laser_rpy" default="0.0 0.0 ${M_PI}" />
+  <xacro:arg name="laser_rpy" default="0.0 0.0 0.0" />
+  <!--xacro:arg name="laser_rpy" default="0.0 0.0 ${M_PI}" /-->
+  <xacro:arg name="laser_xyz" default="0.14 0.0 0.17" />
+  <!--xacro:arg name="laser_xyz" default="0.18 0.12 0.39" /-->
   <xacro:include filename="$(find unicorn_description)/urdf/rplidar_a2.urdf.xacro" />
   <!-- Wheel -->
@@ -176,5 +178,5 @@
       <parent link="chassis_link"/>
       <child link="zed_center"/>
-      <origin xyz="-0.2 0.0 0.3" rpy="0 0 ${-M_PI}"/>
+     <origin xyz="0.14 0.0 0.11" rpy="0 0 ${-M_PI}"/>
     </joint>
   <!-- Orbbec camera -->

Commit message: Reworked files with Joaquin

File: unicorn_description/urdf/unicorn_target.urdf.xacro (robot description, xacro)
@@ -29,5 +29,5 @@
   <xacro:arg name="laser_rpy" default="0.0 0.0 0.0" />
   <!--xacro:arg name="laser_rpy" default="0.0 0.0 ${M_PI}" /-->
-  <xacro:arg name="laser_xyz" default="0.14 0.0 0.17" />
+  <xacro:arg name="laser_xyz" default="-0.14 0.0 0.17" />
   <!--xacro:arg name="laser_xyz" default="0.18 0.12 0.39" /-->
   <xacro:include filename="$(find unicorn_description)/urdf/rplidar_a2.urdf.xacro" />
@@ -178,5 +178,5 @@
       <parent link="chassis_link"/>
       <child link="zed_center"/>
-     <origin xyz="0.14 0.0 0.11" rpy="0 0 ${-M_PI}"/>
+     <origin xyz="-0.14 0.0 0.11" rpy="0 0 ${-M_PI}"/>
     </joint>
   <!-- Orbbec camera -->
@@ -238,5 +238,5 @@
   <ultrasonic_sensor frame="base_ultrasonic_br" topic="br" robot_namespace="$(arg robot_namespace)"/>
   <joint name="ultrasonic_mount_joint_br" type="fixed">
-    <origin xyz="0.45 0.1 0.0" rpy="0 0 0"/>
+    <origin xyz="0.48 0.14 0.0" rpy="0 0 0"/>
     <parent link="chassis_link"/>
     <child link="base_ultrasonic_br" />
@@ -244,5 +244,5 @@
   <ultrasonic_sensor frame="base_ultrasonic_bl" topic="bl" robot_namespace="$(arg robot_namespace)"/>
   <joint name="ultrasonic_mount_joint_bl" type="fixed">
-    <origin xyz="0.45 -0.1 0.0" rpy="0 0 0"/>
+    <origin xyz="0.48 -0.14 0.0" rpy="0 0 0"/>
     <parent link="chassis_link"/>
     <child link="base_ultrasonic_bl" />

Commit message: UWB stuff

File: unicorn_description/urdf/unicorn_target.urdf.xacro (robot description, xacro)
@@ -38,4 +38,7 @@
   <!-- Materials -->
   <xacro:include filename="$(find am_description)/urdf/materials.urdf.xacro" />
+<!-- UWB Tag -->
+  <xacro:arg name="uwb_xyz" default="0.23437 0.0 0.70758" />
+  <xacro:include filename="$(find unicorn_description)/urdf/uwb_tag.urdf.xacro" />
   <link
     name="base_link">
@@ -126,4 +129,11 @@
   <origin xyz="0 0.0 0" rpy="0 0 ${M_PI}" />
   </joint>
+<!-- UWB Joint Marielle -->
+   <uwbtag frame="uwb_tag" robot_namespace="$(arg robot_namespace)"/>
+   <joint name="uwb_chassis_joint" type="fixed">
+      <origin xyz="$(arg uwb_xyz)" rpy= "0.0 0.0 0.0" />
+      <parent link="chassis_link" />
+      <child link="uwb_tag" />
+   </joint>
   <link name="zed_left_camera">
         <visual>

Commit message: Status after testing

File: unicorn_description/urdf/unicorn_target.urdf.xacro (robot description, xacro)
@@ -130,9 +130,9 @@
   </joint>
 <!-- UWB Joint Marielle -->
-   <uwbtag frame="uwb_tag" robot_namespace="$(arg robot_namespace)"/>
+   <uwbtag frame="uwb_t" robot_namespace="$(arg robot_namespace)"/>
    <joint name="uwb_chassis_joint" type="fixed">
-      <origin xyz="$(arg uwb_xyz)" rpy= "0.0 0.0 0.0" />
+      <origin xyz="$(arg uwb_xyz)" rpy= "0.0 0.0 0.0"/>
       <parent link="chassis_link" />
-      <child link="uwb_tag" />
+      <child link="uwb_t" />
    </joint>
   <link name="zed_left_camera">

File: unicorn_description/urdf/uwb_tag.urdf.xacro (robot description, xacro)
@@ -1,10 +1,11 @@
 <?xml version="1.0"?>
 <robot xmlns:xacro="http://www.ros.org/wiki/xacro">
-	<xacro:macro name="uwbtag" params="frame:=uwb_tag robot_namespace:=/" >
+	<xacro:macro name="uwbtag" params="frame:=uwb_t robot_namespace:=/" >
 	   <link name="${frame}">
 	    <visual>
 		<origin xyz = "0.0 0.0 0.0" rpy= "0.0 0.0 0.0" />
 		<geometry>
-			<mesh filename="package://unicorn_description/meshes/UWB.STL" />
+			<!--mesh filename="package://unicorn_description/meshes/UWB.STL" /-->
+			<box size="0.05 0.05 0.05"/>
 		</geometry>
    	    </visual>
